File: DirtyMirrorV2.kicad_pcb (KiCad board)
At the start: 2 copper layers, 50 x 50 mm, 70 parts, among them J1 PWR, J2 ScopeGroundLoop, SW1 SW_SPDT, U1 TL072, U2 TL074, U3 TL074

Commit message: dehiss changes
Parts:
- R10, R7: value 56k -> 51k
- R16, R18: value 47k -> 39k
- R27: value 47k -> 100k
- R28: value 100k -> 47k
- R32: value 12k -> 18k
- R33: value 470k -> 680k
- R5: value 22k -> 33k
- R6: value 560k -> 1M
