File: DirtyMirrorV2.kicad_pcb (KiCad board)
At the start: 2 copper layers, 54 x 58 mm, 72 parts, among them J1 PWR, J3 Power, SW1 SW_SPDT, U1 TL072, U2 TL074, U3 TL074

Commit message: changed switching scheme
Parts:
- J3: moved to B.Cu
Connections:
- C1 pad 2: /Low_In -> 0
- C2 pad 2: /Low_In -> 0
- C4 pad 2: /Low_In -> 0
- D1 pad 2: +9V -> /LED_hi
- J1 pad 3: /Low_In -> /LED_hi
- J1 pad 4: 0 -> +9V
- J2 pad 1: /Low_In -> 0
- J3 pad 1: /Low_In -> 0
- R2 pad 2: /Low_In -> 0
- R36 pad 2: /Low_In -> 0
- U1 pad 4: /Low_In -> 0
Routing:
- net /Low_In: track 120.7 -> 0.00 mm, vias 1 -> 0
- net /LED_hi: track 0.00 -> 89.4 mm, vias 0 -> 1
- net +9V: track 193.3 -> 233.1 mm
- net FX_IN: track 86.8 -> 81.0 mm
- net 0: vias 33 -> 35

Commit message: prettier routing, DRC passing
Parts:
- moved J3 0.48 mm to (35.0, 55.6)
- moved TP3 0.36 mm to (30.9, 50.3)
Routing:
- net +9V: track 233.1 -> 166.3 mm
- net /FxFull: track 54.9 -> 67.3 mm
- net Net-(R26-Pad2): track 17.3 -> 14.4 mm
- net /LED_hi: track 89.4 -> 89.8 mm, vias 1 -> 0
- net 0: vias 35 -> 42
Other:
- board text added: "Rev 3- 08/2026 Hayden Setlik"
- board text removed: "Rev 2- 08/2026 Hayden Setlik"
