File: DirtyMirrorV2.kicad_sch (KiCad schematic)
At the start: 72 parts, among them J1 PWR, J2 ScopeGroundLoop, SW1 SW_SPDT, U1 TL072, U2 TL074, U3 TL074

Commit message: dehiss changes
Parts:
- C6: value 2n2 -> 1n
- R19: value 18k -> 22k
Other:
- moved on the sheet: C11, R16, R17, R18, R20, R21, R22, R23, R24, R26, R30, R31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

Commit message: switched hi-pass back
Parts:
- R3: value 22k -> 4k7
Changed lines of the file:
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@@
 			)
 		)
-		(property "Value" "22k"
+		(property "Value" "4k7"
 			(at 57.15 62.2299 0)
 			(show_name no)

Commit message: more aggressive dehiss
Parts:
- R15: value 18k -> 47k
- R19: value 22k -> 33k
Changed lines of the file:
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@@
 			)
 		)
-		(property "Value" "18k"
+		(property "Value" "47k"
 			(at 241.935 161.29 90)
 			(show_name no)
@@
 			)
 		)
-		(property "Value" "22k"
+		(property "Value" "33k"
 			(at 250.825 161.29 90)
 			(show_name no)

Commit message: folding limits
Parts:
- R10, R7: value 51k -> 56k
- R16, R18: value 39k -> 47k
- R5: value 33k -> 56k
Changed lines of the file:
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@@
 			)
 		)
-		(property "Value" "39k"
+		(property "Value" "47k"
 			(at 250.19 97.79 90)
 			(show_name no)
@@
 			)
 		)
-		(property "Value" "33k"
+		(property "Value" "56k"
 			(at 73.66 46.99 90)
 			(show_name no)
@@
 			)
 		)
-		(property "Value" "51k"
+		(property "Value" "56k"
 			(at 134.62 78.1049 0)
 			(show_name no)
@@
 			)
 		)
-		(property "Value" "51k"
+		(property "Value" "56k"
 			(at 130.81 113.6649 0)
 			(show_name no)
@@
 		(fields_autoplaced yes)
 		(property "Reference" "R16"
-			(at 251.46 78.105 90)
-			(show_name no)
-			(do_not_autoplace no)
-			(effects
-				(font
-					(size 1.27 1.27)
-				)
-			)
-		)
-		(property "Value" "39k"
-			(at 251.46 80.645 90)
-			(show_name no)
-			(do_not_autoplace no)
+			(at 251.46 77.47 90)
+			(show_name no)
+			(do_not_autoplace no)
+			(effects
+				(font
+					(size 1.27 1.27)
+				)
+			)
+		)
+		(property "Value" "47k"
+			(at 251.46 80.01 90)
+			(show_name no)
+			(do_not_autoplace no)
