File: Simulations/ToneStackSim/ToneStackSim.kicad_sch (KiCad schematic)
At the start: 9 parts

Commit message: switched hi-pass back
Parts:
- added C11: 2u2, Capacitor_SMD:C_0805_2012Metric, symbol Device:C
- added C12: 10n, Capacitor_SMD:C_0805_2012Metric, symbol Device:C
- added C13: 100n, Capacitor_SMD:C_0805_2012Metric, symbol Device:C
- added R2: Potentiometer, symbol Simulation_SPICE:Potentiometer
- added R30: 47k, Resistor_SMD:R_0805_2012Metric, symbol Device:R_US
- added R31: 100k, Resistor_SMD:R_0805_2012Metric, symbol Device:R_US
- added R33: 4k7, Resistor_SMD:R_0805_2012Metric, symbol Device:R_US
- added R34: 27k, Resistor_SMD:R_0805_2012Metric, symbol Device:R_US
- added V2: VSIN, symbol Simulation_SPICE:VSIN
Connections:
- net 0: now also C13.2, R31.2, R34.2, V2.2
- net Dry: now reaches R27.2, R28.1
- net HiPass renamed HP1
- net In: no longer names the net of C8.1, C9.1, V1.1
- net LowPass renamed LP1
- net Out renamed Out1
- new net: C11.1, C12.1, V2.1
- new net: R30.2, R31.1
- new net: C11.2, R30.1, R33.1
- new net HP2: C12.2, R2.1, R34.1
- new net LP2: C13.1, R2.3, R33.2
- new net Out2: R2.2
