File: Simulations/DeHissFilterSim/DeHissFilterSim.kicad_sch (KiCad schematic)
At the start: 15 parts, among them U1 TL072, U2 TL072

Commit message: more aggressive dehiss
Parts:
- R15: value 18k -> 47k
- R16: value 33k -> 18k
- R19: value 22k -> 33k
- R20: value 33k -> 22k
Changed lines of the file:
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@@
 		(fields_autoplaced yes)
 		(property "Reference" "R16"
-			(at 77.47 42.545 90)
-			(show_name no)
-			(do_not_autoplace no)
-			(effects
-				(font
-					(size 1.27 1.27)
-				)
-			)
-		)
-		(property "Value" "33k"
-			(at 77.47 45.085 90)
+			(at 77.47 41.91 90)
+			(show_name no)
+			(do_not_autoplace no)
+			(effects
+				(font
+					(size 1.27 1.27)
+				)
+			)
+		)
+		(property "Value" "18k"
+			(at 77.47 44.45 90)
 			(show_name no)
 			(do_not_autoplace no)
@@
 			)
 		)
-		(property "Value" "22k"
+		(property "Value" "33k"
 			(at 86.36 92.71 90)
 			(show_name no)
@@
 		(fields_autoplaced yes)
 		(property "Reference" "R20"
-			(at 86.36 42.545 90)
-			(show_name no)
-			(do_not_autoplace no)
-			(effects
-				(font
-					(size 1.27 1.27)
-				)
-			)
-		)
-		(property "Value" "33k"
-			(at 86.36 45.085 90)
+			(at 86.36 41.91 90)
+			(show_name no)
+			(do_not_autoplace no)
+			(effects
+				(font
+					(size 1.27 1.27)
+				)
+			)
+		)
+		(property "Value" "22k"
+			(at 86.36 44.45 90)
 			(show_name no)
 			(do_not_autoplace no)
@@
 			)
 		)
-		(property "Value" "18k"
+		(property "Value" "47k"
 			(at 77.47 92.71 90)
 			(show_name no)
